File: kicad project/nearness intellijel 1u.kicad_sch (KiCad schematic)
At the start: 48 parts, among them J1 PJ301M12, J10 PJ301M12, J2 PJ301M12, J3 PJ301M12, J4 PJ301M12, J5 PJ301M12, J6 PJ301M12, J7 PJ301M12, J8 PJ301M12, J9 PJ301M12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

Commit message: Adjusted resistor values
Parts:
- D1, D2: value 1N5819HW -> Schottky
- R11, R4: value 439k -> 442k
- R12, R3: value 103k -> 102k
- R13, R2: value 1M67 -> 1M65
- R25, R26, R7, R8: value 141k -> 140k
